Commit message: feat: add separable gripper and pick place demo for B601-RS fix: remove redundant configuration files

File: src/rebotarm_bringup/description/urdf/00-arm-rs_asm-v3.urdf (robot description, URDF)
Before this commit: robot 00-arm-rs_asm-v3, 10 links, 9 joints
Joints:
- removed joint joint_left
- removed joint joint_right
- added joint gripper_joint1: type prismatic, parent gripper_end, child gripper_left, origin xyz=-0.041939 -7.3385E-05 0 rpy=1.5708 -1.5708 0, axis 0 0 1, limit lower=0 upper=0.05 effort=500 velocity=10
- added joint gripper_joint2: type prismatic, parent gripper_end, child gripper_right, origin xyz=-0.041939 7.3385E-05 0 rpy=-1.5708 -1.5708 0, axis 0 0 1, limit lower=0 upper=0.0715 effort=500 velocity=10

File: src/rebotarm_moveit_config/config/rebotarm_rs.ros2_control.xacro (robot description, xacro)
@@ -61,4 +61,22 @@
         </state_interface>
       </joint>
+      <joint name="gripper_joint1">
+        <command_interface name="position"/>
+        <state_interface name="position">
+          <param name="initial_value">${initial_positions['gripper_joint1']}</param>
+        </state_interface>
+        <state_interface name="velocity">
+          <param name="initial_value">0.0</param>
+        </state_interface>
+      </joint>
+      <joint name="gripper_joint2">
+        <command_interface name="position"/>
+        <state_interface name="position">
+          <param name="initial_value">${initial_positions['gripper_joint2']}</param>
+        </state_interface>
+        <state_interface name="velocity">
+          <param name="initial_value">0.0</param>
+        </state_interface>
+      </joint>
     </ros2_control>
   </xacro:macro>
